File: onstep-ramps-shield.kicad_pcb (KiCad board)
At the start: 2 copper layers, 114.3 x 67.3 mm, 29 parts

Commit message: Copper fill
Routing:
- net E0_2B: track 129.3 -> 128.5 mm
- added copper zone on B.Cu, net (none)
- added copper zone on F.Cu, net (none)
Changed lines of the file:
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@@
     (thickness 1.6002)
     (drawings 29)
-    (tracks 487)
+    (tracks 486)
     (zones 0)
     (modules 29)
@@
       (drillshape 0)
       (scaleselection 1)
-      (outputdirectory "./gerbers_for_aisler"))
+      (outputdirectory "./gerbers"))
   )
   (net 0 "")
@@
     (add_net "Net-(D1-Pad2)")
     (add_net "Net-(D2-Pad2)")
-    (add_net "Net-(DEC1-Pad5)")
-    (add_net "Net-(DEC1-Pad6)")
-    (add_net "Net-(FOC1-Pad5)")
-    (add_net "Net-(FOC1-Pad6)")
-    (add_net "Net-(FOC2-Pad5)")
-    (add_net "Net-(FOC2-Pad6)")
-    (add_net "Net-(J_AUX1-Pad1)")
-    (add_net "Net-(J_AUX1-Pad2)")
-    (add_net "Net-(J_AUX1-Pad3)")
-    (add_net "Net-(J_AUX1-Pad4)")
-    (add_net "Net-(J_AUX1-Pad6)")
-    (add_net "Net-(J_AUX1-Pad7)")
-    (add_net "Net-(J_AUX1-Pad8)")
-    (add_net "Net-(J_AUX2-Pad1)")
-    (add_net "Net-(J_AUX2-Pad10)")
-    (add_net "Net-(J_AUX2-Pad2)")
-    (add_net "Net-(J_AUX2-Pad3)")
-    (add_net "Net-(J_AUX2-Pad4)")
-    (add_net "Net-(J_AUX2-Pad5)")
-    (add_net "Net-(J_AUX2-Pad6)")
-    (add_net "Net-(J_AUX2-Pad7)")
-    (add_net "Net-(J_AUX2-Pad8)")
-    (add_net "Net-(J_AUX2-Pad9)")
-    (add_net "Net-(J_AUX3-Pad1)")
-    (add_net "Net-(J_AUX3-Pad2)")
-    (add_net "Net-(J_AUX3-Pad3)")
-    (add_net "Net-(J_AUX3-Pad4)")
-    (add_net "Net-(J_AUX3-Pad5)")
-    (add_net "Net-(J_AUX3-Pad6)")
-    (add_net "Net-(J_AUX3-Pad7)")
-    (add_net "Net-(J_AUX3-Pad8)")
-    (add_net "Net-(J_AUX4-Pad10)")
-    (add_net "Net-(J_AUX4-Pad11)")
-    (add_net "Net-(J_AUX4-Pad12)")
-    (add_net "Net-(J_AUX4-Pad13)")
-    (add_net "Net-(J_AUX4-Pad14)")
-    (add_net "Net-(J_AUX4-Pad15)")
-    (add_net "Net-(J_AUX4-Pad16)")
-    (add_net "Net-(J_AUX4-Pad17)")
-    (add_net "Net-(J_AUX4-Pad18)")
-    (add_net "Net-(J_AUX4-Pad3)")
-    (add_net "Net-(J_AUX4-Pad4)")
-    (add_net "Net-(J_AUX4-Pad5)")
-    (add_net "Net-(J_AUX4-Pad6)")
-    (add_net "Net-(J_AUX4-Pad7)")
-    (add_net "Net-(J_AUX4-Pad8)")
-    (add_net "Net-(J_AUX4-Pad9)")
-    (add_net "Net-(J_RET1-PadR)")
     (add_net "Net-(J_RET1-PadS)")
-    (add_net "Net-(J_SERV1-Pad2)")
-    (add_net "Net-(J_SERV2-Pad2)")
-    (add_net "Net-(J_SERV3-Pad1)")
-    (add_net "Net-(J_SERV3-Pad2)")
-    (add_net "Net-(J_SERV4-Pad1)")
-    (add_net "Net-(J_SERV4-Pad2)")
-    (add_net "Net-(RA1-Pad5)")
-    (add_net "Net-(RA1-Pad6)")
     (add_net PEC1)
     (add_net RETICULE_LED1)
@@
   (segment (start 181.61 60.96) (end 186.69 55.88) (width 0.5) (layer Back) (net 5))
   (segment (start 181.61 63.5) (end 181.61 60.96) (width 0.5) (layer Back) (net 5))
-  (segment (start 147.686023 51.5899) (end 146.936012 52.339911) (width 0.5) (layer Front) (net 5))
-  (segment (start 154.573977 51.5899) (end 147.686023 51.5899) (width 0.5) (layer Front) (net 5))
-  (segment (start 101.310034 56.089966) (end 93.98 63.42) (width 0.5) (layer Front) (net 5))
-  (segment (start 146.936012 52.339911) (end 118.677389 52.339911) (width 0.5) (layer Front) (net 5))
-  (segment (start 166.484077 63.5) (end 154.573977 51.5899) (width 0.5) (layer Front) (net 5))
-  (segment (start 181.61 63.5) (end 166.484077 63.5) (width 0.5) (layer Front) (net 5))
-  (segment (start 114.927334 56.089966) (end 101.310034 56.089966) (width 0.5) (layer Front) (net 5))
-  (segment (start 118.677389 52.339911) (end 114.927334 56.089966) (width 0.5) (layer Front) (net 5))
-  (segment (start 93.98 63.42) (end 93.98 64.77) (width 0.5) (layer Front) (net 5))
+  (segment (start 166.484077 63.5) (end 181.61 63.5) (width 0.5) (layer Front) (net 5))
+  (segment (start 154.573977 51.5899) (end 166.484077 63.5) (width 0.5) (layer Front) (net 5))
+  (segment (start 147.686023 51.5899) (end 154.573977 51.5899) (width 0.5) (layer Front) (net 5))
+  (segment (start 118.677389 52.339911) (end 146.936012 52.339911) (width 0.5) (layer Front) (net 5))
+  (segment (start 114.927334 56.089966) (end 118.677389 52.339911) (width 0.5) (layer Front) (net 5))
+  (segment (start 146.936012 52.339911) (end 147.686023 51.5899) (width 0.5) (layer Front) (net 5))
+  (segment (start 102.660034 56.089966) (end 114.927334 56.089966) (width 0.5) (layer Front) (net 5))
+  (segment (start 93.98 64.77) (end 102.660034 56.089966) (width 0.5) (layer Front) (net 5))
   (via (at 181.61 64.77) (size 0.8) (drill 0.4) (layers Front Back) (net 6))
   (segment (start 190.5 57.15) (end 192.289989 58.939989) (width 0.5) (layer Back) (net 6))
@@
   (segment (start 160.101404 64.768596) (end 165.1 59.77) (width 0.5) (layer Back) (net 34))
   (segment (start 156.211404 64.768596) (end 160.101404 64.768596) (width 0.5) (layer Back) (net 34))
+  (zone (net 0) (net_name "") (layer Front) (hatch edge 0.508)
+    (connect_pads (clearance 0.508))
+    (min_thickness 0.254)
+    (fill yes (arc_segments 32) (thermal_gap 0.508) (thermal_bridge_width 0.508) (smoothing chamfer))
+    (polygon
+      (pts
+        (xy 201.93 53.34) (xy 201.93 115.57) (xy 200.66 116.84) (xy 91.44 116.84) (xy 90.17 115.57)
+        (xy 90.17 110.49) (xy 91.44 109.22) (xy 137.16 109.22) (xy 139.7 106.68) (xy 139.7 92.71)
+        (xy 137.16 90.17) (xy 91.44 90.17) (xy 90.17 88.9) (xy 90.17 87.63) (xy 91.44 86.36)
+        (xy 135.89 86.36) (xy 137.16 86.36) (xy 139.7 83.82) (xy 139.7 67.31) (xy 138.43 66.04)
+        (xy 91.44 66.04) (xy 90.17 64.77) (xy 90.17 53.34) (xy 91.44 52.07) (xy 200.66 52.07)
+      )
+    )
+  )
+  (zone (net 0) (net_name "") (layer Back) (hatch edge 0.508)
+    (connect_pads (clearance 0.508))
+    (min_thickness 0.254)
+    (fill yes (arc_segments 32) (thermal_gap 0.508) (thermal_bridge_width 0.508))
+    (polygon
+      (pts
+        (xy 201.93 53.34) (xy 201.93 115.57) (xy 200.66 116.84) (xy 91.44 116.84) (xy 90.17 115.57)
+        (xy 90.17 110.49) (xy 91.44 109.22) (xy 137.16 109.22) (xy 139.7 106.68) (xy 139.7 92.71)
+        (xy 137.16 90.17) (xy 91.44 90.17) (xy 90.17 88.9) (xy 90.17 87.63) (xy 91.44 86.36)
+        (xy 135.89 86.36) (xy 137.16 86.36) (xy 139.7 83.82) (xy 139.7 67.31) (xy 138.43 66.04)
+        (xy 91.44 66.04) (xy 90.17 64.77) (xy 90.17 53.34) (xy 91.44 52.07) (xy 200.66 52.07)
+      )
+    )
+  )
 )
